File: pcb/Pinky2.sch (KiCad schematic (older format))
At the start: 22 parts, among them SW1 RESET_SW, SW10 SW_PUSH, SW11 SW_PUSH, SW2 SW_PUSH, SW3 SW_PUSH, SW4 SW_PUSH, SW5 SW_PUSH, SW6 SW_PUSH, SW7 SW_PUSH, SW8 SW_PUSH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

Commit message: initial commit
Parts:
- added D10, D11, D12: D, kbd:D3_TH_SMD, symbol Device:D
- added SW12, SW13: SW_PUSH, kbd:CherryMX_Hotswap, symbol Pinky2-rescue:SW_PUSH-kbd-Pinky3-rescue
- added SW8: SW_PUSH, lib:Choc_Hotswap, symbol Pinky2-rescue:SW_PUSH-kbd-Pinky3-rescue
- renumbered D10 to D13, SW8 to SW11, SW11 to SW14
Connections:
- net col2: now also SW8.1; no longer SW11.1
- net col3: now also SW11.1; no longer SW14.1
- net row0: now also D11.1 (K)
- net row1: now also D12.1 (K)
- net row2: now also D10.1 (K)
- net col4: now reaches U1.16 (B1)
- net col4: now also SW14.1, SW12.2, SW13.1
- net at SW11.2: now also D10.2 (A); no longer D7.2 (A)
- new net: D11.2 (A), SW12.1
- new net: D12.2 (A), SW13.2
- new net: D7.2 (A), SW8.2
- no-connect marks 12 -> 11
Other:
- moved on the sheet: D13, SW11, SW14
Changed lines of the file:
@@
 $EndComp
 $Comp
-L Pinky2-rescue:SW_PUSH-kbd-Pinky3-rescue SW11
+L Pinky2-rescue:SW_PUSH-kbd-Pinky3-rescue SW14
 U 1 1 5BDC1338
-P 8460 5570
-F 0 "SW11" H 8460 5825 50  0000 C CNN
-F 1 "SW_PUSH" H 8460 5734 50  0000 C CNN
-F 2 "lib:Choc_Hotswap" H 8460 5570 50  0001 C CNN
-F 3 "" H 8460 5570 50  0000 C CNN
-	1    8460 5570
+P 9295 5570
+F 0 "SW14" H 9295 5825 50  0000 C CNN
+F 1 "SW_PUSH" H 9295 5734 50  0000 C CNN
+F 2 "lib:Choc_Hotswap" H 9295 5570 50  0001 C CNN
+F 3 "" H 9295 5570 50  0000 C CNN
+	1    9295 5570
 	1    0    0    -1
 $EndComp
@@
 Text GLabel 4330 5210 0    50   Input ~ 0
 row1
-Text GLabel 4335 5870 0    50   Input ~ 0
-row2
 $Comp
 L Device:D D3
@@
 $EndComp
 $Comp
-L Device:D D10
+L Device:D D13
 U 1 1 5BDFE4ED
-P 8760 5720
-F 0 "D10" V 8806 5641 50  0000 R CNN
-F 1 "D" V 8715 5641 50  0000 R CNN
-F 2 "kbd:D3_TH_SMD" H 8760 5720 50  0001 C CNN
-F 3 "~" H 8760 5720 50  0001 C CNN
-	1    8760 5720
+P 9595 5720
+F 0 "D13" V 9641 5641 50  0000 R CNN
+F 1 "D" V 9550 5641 50  0000 R CNN
+F 2 "kbd:D3_TH_SMD" H 9595 5720 50  0001 C CNN
+F 3 "~" H 9595 5720 50  0001 C CNN
+	1    9595 5720
 	0    -1   -1   0
 $EndComp
@@
 	7305 4230 7305 4910
 Wire Wire Line
-	7905 5210 8760 5210
-Connection ~ 7905 5210
-Wire Wire Line
 	8160 4230 8160 4910
 Wire Wire Line
 	7905 4530 8760 4530
-Connection ~ 8160 4910
-Wire Wire Line
-	8160 4910 8160 5570
 Connection ~ 7030 5210
 Connection ~ 7030 4530
@@
 	8160 3635 8160 4230
 Wire Wire Line
-	4335 5870 7905 5870
-Wire Wire Line
 	4320 4530 6140 4530
 Wire Wire Line
@@
 Text GLabel 2605 1945 2    50   Input ~ 0
 col1
-NoConn ~ 2605 2245
 NoConn ~ 2605 2345
 NoConn ~ 2605 2445
 NoConn ~ 1205 2545
-$Comp
-L Device:D D7
-U 1 1 5D97877F
-P 7905 5720
-F 0 "D7" V 7951 5641 50  0000 R CNN
-F 1 "D" V 7860 5641 50  0000 R CNN
-F 2 "kbd:D3_TH_SMD" H 7905 5720 50  0001 C CNN
-F 3 "~" H 7905 5720 50  0001 C CNN
-	1    7905 5720
-	0    -1   -1   0
-$EndComp
 $Comp
 L Pinky2-rescue:SW_PUSH-kbd-Pinky3-rescue SW7
@@
 $EndComp
 $Comp
+L Pinky2-rescue:SW_PUSH-kbd-Pinky3-rescue SW11
+U 1 1 5D97788B
+P 8460 5570
+F 0 "SW11" H 8460 5825 50  0000 C CNN
+F 1 "SW_PUSH" H 8460 5734 50  0000 C CNN
+F 2 "lib:Choc_Hotswap" H 8460 5570 50  0001 C CNN
+F 3 "" H 8460 5570 50  0000 C CNN
+	1    8460 5570
+	1    0    0    -1
+$EndComp
+Wire Wire Line
+	8160 4910 8160 5570
+NoConn ~ 1205 1845
+NoConn ~ 1205 1945
+NoConn ~ 1205 2345
+NoConn ~ 1205 2445
+$Comp
+L Pinky2-rescue:SW_PUSH-kbd-Pinky3-rescue SW13
+U 1 1 5D9CD1F4
+P 9295 4910
+F 0 "SW13" H 9295 5165 50  0000 C CNN
+F 1 "SW_PUSH" H 9295 5074 50  0000 C CNN
+F 2 "kbd:CherryMX_Hotswap" H 9295 4910 50  0001 C CNN
+F 3 "" H 9295 4910 50  0000 C CNN
+	1    9295 4910
+	1    0    0    -1
+$EndComp
+$Comp
+L Device:D D11
+U 1 1 5D9CD1FA
+P 9595 4380
+F 0 "D11" V 9641 4301 50  0000 R CNN
+F 1 "D" V 9550 4301 50  0000 R CNN
+F 2 "kbd:D3_TH_SMD" H 9595 4380 50  0001 C CNN
+F 3 "~" H 9595 4380 50  0001 C CNN
+	1    9595 4380
+	0    -1   -1   0
+$EndComp
+Connection ~ 8160 4910
+Text GLabel 8995 3655 1    50   Input ~ 0
+col4
+$Comp
+L Device:D D12
+U 1 1 5D9CD200
+P 9595 5060
+F 0 "D12" V 9641 4981 50  0000 R CNN
+F 1 "D" V 9550 4981 50  0000 R CNN
+F 2 "kbd:D3_TH_SMD" H 9595 5060 50  0001 C CNN
+F 3 "~" H 9595 5060 50  0001 C CNN
+	1    9595 5060
+	0    -1   -1   0
+$EndComp
+Connection ~ 7905 5210
+Wire Wire Line
+	7905 5210 8760 5210
+Wire Wire Line
+	8760 5210 9595 5210
+Connection ~ 8760 5210
+Wire Wire Line
+	8760 4530 9595 4530
+Connection ~ 8760 4530
+Wire Wire Line
+	8995 3655 8995 4230
+Wire Wire Line
+	8995 4230 8995 4910
+Connection ~ 8995 4230
+Wire Wire Line
+	8995 4910 8995 5570
+Connection ~ 8995 4910
+$Comp
+L Pinky2-rescue:SW_PUSH-kbd-Pinky3-rescue SW12
+U 1 1 5D9CD1EE
+P 9295 4230
+F 0 "SW12" H 9295 4485 50  0000 C CNN
+F 1 "SW_PUSH" H 9295 4394 50  0000 C CNN
+F 2 "kbd:CherryMX_Hotswap" H 9295 4230 50  0001 C CNN
+F 3 "" H 9295 4230 50  0000 C CNN
+	1    9295 4230
+	-1   0    0    -1
+$EndComp
+Text GLabel 4335 5870 0    50   Input ~ 0
+row2
+Text GLabel 2605 2245 2    50   Input ~ 0
+col4
+Wire Wire Line
+	8760 5870 9595 5870
+$Comp
+L Device:D D10
+U 1 1 5DA03BD1
+P 8760 5720
+F 0 "D10" V 8806 5641 50  0000 R CNN
+F 1 "D" V 8715 5641 50  0000 R CNN
+F 2 "kbd:D3_TH_SMD" H 8760 5720 50  0001 C CNN
+F 3 "~" H 8760 5720 50  0001 C CNN
+	1    8760 5720
+	0    -1   -1   0
+$EndComp
+Wire Wire Line
+	4335 5870 7905 5870
+Connection ~ 8760 5870
+$Comp
 L Pinky2-rescue:SW_PUSH-kbd-Pinky3-rescue SW8
-U 1 1 5D97788B
+U 1 1 5DA07CE1
 P 7605 5570
 F 0 "SW8" H 7605 5825 50  0000 C CNN
@@
 	1    0    0    -1
 $EndComp
+$Comp
+L Device:D D7
+U 1 1 5DA07CE7
+P 7905 5720
+F 0 "D7" V 7951 5641 50  0000 R CNN
+F 1 "D" V 7860 5641 50  0000 R CNN
+F 2 "kbd:D3_TH_SMD" H 7905 5720 50  0001 C CNN
+F 3 "~" H 7905 5720 50  0001 C CNN
+	1    7905 5720
+	0    -1   -1   0
+$EndComp
 Wire Wire Line
 	7305 4910 7305 5570
@@
 Wire Wire Line
 	7905 5870 8760 5870
-NoConn ~ 1205 1845
-NoConn ~ 1205 1945
-NoConn ~ 1205 2345
-NoConn ~ 1205 2445
 $EndSCHEMATC
