File: pcb/Pinky2.kicad_pcb (KiCad board)
At the start: 2 copper layers, 79.4 x 66.3 mm, 31 parts, among them SW1 RESET_SW, SW10 SW_PUSH, SW11 SW_PUSH, SW2 SW_PUSH, SW3 SW_PUSH, SW4 SW_PUSH, SW5 SW_PUSH, SW6 SW_PUSH, SW7 SW_PUSH, SW8 SW_PUSH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

Commit message: initial commit
Parts:
- added D11: D, kbd:D3_TH_SMD, F.Cu at (145.9, 95.0)
- added D12: D, kbd:D3_TH_SMD, F.Cu at (145.9, 98.0)
- added D13: D, kbd:D3_TH_SMD, F.Cu at (106.5, 147.8)
- added SW12: SW_PUSH, kbd:CherryMX_Hotswap, F.Cu at (145.5, 87.2)
- added SW13: SW_PUSH, kbd:CherryMX_Hotswap, F.Cu at (145.6, 106.3)
- added SW14: SW_PUSH, lib:Choc_Hotswap, F.Cu at (152.0, 133.7)
- U1: footprint lib:ProMicro_v2 -> kbd:ProMicro_v2
- moved D10 28.2 mm to (116.5, 145.1), turned to 0 degrees
- moved D7 26.9 mm to (106.5, 145.1)
- moved SW8 7.49 mm to (111.6, 133.7)
- moved SW11 5.83 mm to (131.8, 133.7), turned to 180 degrees
Connections:
- U1 pad 16: Net-(U1-Pad16) -> col4
Routing:
- net reset: track 79.0 -> 18.8 mm
- net col2: track 152.3 -> 110.4 mm
- net col3: track 157.3 -> 118.6 mm, vias 6 -> 4
- net Net-(D10-Pad2): track 26.5 -> 0.00 mm, vias 1 -> 0
- net row2: track 66.8 -> 43.2 mm
- net Net-(D7-Pad2): track 27.1 -> 4.07 mm, vias 1 -> 0
- net col4: track 0.00 -> 14.4 mm, vias 0 -> 1
- net Net-(U1-Pad16): track 14.4 -> 0.00 mm, vias 1 -> 0
- net GND: track 96.3 -> 91.5 mm, vias 16 -> 14
- net (no net): vias 0 -> 1
- removed copper zone on B.Cu, net GND
- removed copper zone on F.Cu, net GND
Other:
- board size 79.4 x 66.3 mm -> 75.3 x 63 mm

Commit message: may be finished pcb
Parts:
- U1: footprint kbd:ProMicro_v2 -> lib:ProMicro_v2
- moved D13 47.9 mm to (148.6, 125.0), turned to 340 degrees
- moved D10 28.2 mm to (129.8, 120.3), turned to 350 degrees
- moved D7 26.9 mm to (108.2, 118.3)
- moved Ref** 20.8 mm to (134.4, 116.0)
- moved SW1 19.9 mm to (149.6, 121.7), turned to 160 degrees
- moved Ref** 19.5 mm to (135.1, 95.7)
- moved SW8 7.49 mm to (108.2, 127.0)
- moved SW11 5.83 mm to (128.4, 128.9), turned to 170 degrees
- moved SW14 3.95 mm to (148.0, 134.1), turned to 160 degrees
- moved D11 3.31 mm to (145.2, 98.2)
- moved D12 2.89 mm to (145.2, 100.8)
- moved SW12 2.84 mm to (145.2, 90.0)
- moved SW13 2.78 mm to (145.2, 109.1)
Connections:
- SW12 pad 1: Net-(D11-Pad2) -> col4
- SW12 pad 2: col4 -> Net-(D11-Pad2)
Routing:
- net col4: track 14.4 -> 177.0 mm, vias 1 -> 7
- net reset: track 18.8 -> 99.6 mm
- net row2: track 43.2 -> 90.1 mm
- net col2: track 110.4 -> 150.2 mm
- net col3: track 118.6 -> 155.2 mm, vias 4 -> 5
- net Net-(D11-Pad2): track 0.00 -> 33.1 mm, vias 0 -> 1
- net Net-(D10-Pad2): track 0.00 -> 27.8 mm, vias 0 -> 1
- net Net-(D13-Pad2): track 0.00 -> 27.5 mm, vias 0 -> 1
- net row1: track 109.9 -> 133.4 mm
- net Net-(D7-Pad2): track 4.07 -> 26.9 mm, vias 0 -> 1
- net GND: track 91.5 -> 114.1 mm, vias 14 -> 42
- net row0: track 125.8 -> 148.5 mm
- net Net-(D12-Pad2): track 0.00 -> 16.8 mm
- net (no net): vias 1 -> 0
- added copper zone on B.Cu, net GND
- added copper zone on F.Cu, net GND
Other:
- board size 75.3 x 63 mm -> 100 x 72.7 mm

Commit message: design finished
Parts:
- removed ? (x2): , 
Routing:
- net col4: vias 7 -> 6
- net GND: vias 42 -> 47
