File: bottom-plate/Pinky2-bottom-plate.kicad_pcb (KiCad board)
At the start: 2 copper layers, 79.4 x 66.3 mm, 3 parts

Commit message: design finished
Parts:
- moved Ref** 20.8 mm to (134.4, 116.0)
- moved Ref** 19.5 mm to (135.1, 95.7)
Other:
- board size 79.4 x 66.3 mm -> 100 x 72.7 mm
Changed lines of the file:
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@@
   (page A4)
   (title_block
-    (title "Pinky2 Bottom Plate")
-    (date 2019-10-06)
+    (title "Pinky2 bottom plate")
+    (date 2019-10-09)
     (rev 1.0)
     (company @tamanishi)
@@
     (mod_text_size 1 1)
     (mod_text_width 0.15)
-    (pad_size 5 5)
-    (pad_drill 4.8)
+    (pad_size 2.3 2)
+    (pad_drill 0)
     (pad_to_mask_clearance 0.2)
     (solder_mask_min_width 0.25)
@@
   )
   (module kbd:HOLE_M2 (layer F.Cu)
-    (at 116 91.9)
+    (at 135.1 95.725)
     (fp_text reference Ref** (at 0 -3.2) (layer F.Fab)
       (effects (font (size 1 1) (thickness 0.15)))
@@
   )
   (module kbd:HOLE_M2 (layer F.Cu)
-    (at 114 112.1)
+    (at 134.425 116.05)
     (fp_text reference Ref** (at 0 -3.2) (layer F.Fab)
       (effects (font (size 1 1) (thickness 0.15)))
@@
       (clearance 0.85))
   )
-  (dimension 66.3 (width 0.3) (layer F.CrtYd)
-    (gr_text "66.300 mm" (at 54.824901 106.5 90) (layer F.CrtYd)
+  (dimension 72.79 (width 0.3) (layer F.CrtYd)
+    (gr_text "72.790 mm" (at 55.7 109.745 270) (layer F.CrtYd)
       (effects (font (size 1.5 1.5) (thickness 0.3)))
     )
-    (feature1 (pts (xy 60.05 73.35) (xy 56.33848 73.35)))
-    (feature2 (pts (xy 60.05 139.65) (xy 56.33848 139.65)))
-    (crossbar (pts (xy 56.924901 139.65) (xy 56.924901 73.35)))
-    (arrow1a (pts (xy 56.924901 73.35) (xy 57.511322 74.476504)))
-    (arrow1b (pts (xy 56.924901 73.35) (xy 56.33848 74.476504)))
-    (arrow2a (pts (xy 56.924901 139.65) (xy 57.511322 138.523496)))
-    (arrow2b (pts (xy 56.924901 139.65) (xy 56.33848 138.523496)))
+    (feature1 (pts (xy 60.1 146.14) (xy 57.213579 146.14)))
+    (feature2 (pts (xy 60.1 73.35) (xy 57.213579 73.35)))
+    (crossbar (pts (xy 57.8 73.35) (xy 57.8 146.14)))
+    (arrow1a (pts (xy 57.8 146.14) (xy 57.213579 145.013496)))
+    (arrow1b (pts (xy 57.8 146.14) (xy 58.386421 145.013496)))
+    (arrow2a (pts (xy 57.8 73.35) (xy 57.213579 74.476504)))
+    (arrow2b (pts (xy 57.8 73.35) (xy 58.386421 74.476504)))
   )
-  (dimension 78.45 (width 0.3) (layer F.CrtYd)
-    (gr_text "78.450 mm" (at 99.275 69.149999) (layer F.CrtYd)
+  (gr_line (start 136 139.75) (end 153.125 146.025) (layer Edge.Cuts) (width 0.15))
+  (gr_line (start 116.5 136.3) (end 136 139.75) (layer Edge.Cuts) (width 0.15))
+  (gr_line (start 60.75 136.3) (end 116.5 136.3) (layer Edge.Cuts) (width 0.15))
+  (gr_line (start 160.000347 128.974287) (end 153.944883 145.672519) (layer Edge.Cuts) (width 0.15))
+  (gr_arc (start 153.331265 145.375) (end 153.125 146.025) (angle -81.73893252) (layer Edge.Cuts) (width 0.15))
+  (gr_arc (start 159.352828 128.762905) (end 160.000347 128.974287) (angle -82.21241903) (layer Edge.Cuts) (width 0.15))
+  (gr_line (start 154.25 126.175) (end 159.65 128.15) (layer Edge.Cuts) (width 0.15))
+  (gr_line (start 154.25 81.468823) (end 154.25 126.175) (layer Edge.Cuts) (width 0.15))
+  (dimension 100 (width 0.3) (layer F.CrtYd)
+    (gr_text "100.000 mm" (at 110.05 68.675) (layer F.CrtYd)
       (effects (font (size 1.5 1.5) (thickness 0.3)))
     )
-    (feature1 (pts (xy 138.5 73.4) (xy 138.5 70.663578)))
-    (feature2 (pts (xy 60.05 73.4) (xy 60.05 70.663578)))
-    (crossbar (pts (xy 60.05 71.249999) (xy 138.5 71.249999)))
-    (arrow1a (pts (xy 138.5 71.249999) (xy 137.373496 71.83642)))
-    (arrow1b (pts (xy 138.5 71.249999) (xy 137.373496 70.663578)))
-    (arrow2a (pts (xy 60.05 71.249999) (xy 61.176504 71.83642)))
-    (arrow2b (pts (xy 60.05 71.249999) (xy 61.176504 70.663578)))
+    (feature1 (pts (xy 160.05 73.4) (xy 160.05 70.188579)))
+    (feature2 (pts (xy 60.05 73.4) (xy 60.05 70.188579)))
+    (crossbar (pts (xy 60.05 70.775) (xy 160.05 70.775)))
+    (arrow1a (pts (xy 160.05 70.775) (xy 158.923496 71.361421)))
+    (arrow1b (pts (xy 160.05 70.775) (xy 158.923496 70.188579)))
+    (arrow2a (pts (xy 60.05 70.775) (xy 61.176504 71.361421)))
+    (arrow2b (pts (xy 60.05 70.775) (xy 61.176504 70.188579)))
   )
   (gr_line (start 98.1 73.35) (end 116.2 73.35) (layer Edge.Cuts) (width 0.15))
-  (gr_arc (start 138.616634 121.852497) (end 139.466634 122.047112) (angle -90.75712949) (layer Edge.Cuts) (width 0.15))
-  (gr_line (start 138.8 121) (end 135.3 120.4) (layer Edge.Cuts) (width 0.15))
-  (gr_line (start 116.1 136.3) (end 60.75 136.3) (layer Edge.Cuts) (width 0.15))
-  (gr_line (start 116.1 136.3) (end 117.4 136.3) (layer Edge.Cuts) (width 0.15))
   (gr_arc (start 61.055846 79.743142) (end 60.9 78.743143) (angle -73.04255484) (layer Edge.Cuts) (width 0.15))
-  (gr_arc (start 134.5 77.693735) (end 135.3 77.693823) (angle -82.8313174) (layer Edge.Cuts) (width 0.15))
-  (gr_arc (start 135.790389 138.9) (end 135.640389 139.6) (angle -94.50009784) (layer Edge.Cuts) (width 0.15))
+  (gr_arc (start 153.45 81.468735) (end 154.25 81.468823) (angle -82.8313174) (layer Edge.Cuts) (width 0.15))
   (gr_arc (start 60.75 135.6) (end 60.05 135.6) (angle -90) (layer Edge.Cuts) (width 0.15))
-  (gr_line (start 117.4 136.3) (end 135.640389 139.6) (layer Edge.Cuts) (width 0.15))
-  (gr_line (start 139.466634 122.047112) (end 136.5 138.994615) (layer Edge.Cuts) (width 0.15))
-  (gr_line (start 135.3 77.693823) (end 135.3 120.4) (layer Edge.Cuts) (width 0.15))
-  (gr_line (start 116.2 73.35) (end 134.6 76.9) (layer Edge.Cuts) (width 0.15))
+  (gr_line (start 116.2 73.35) (end 153.54992 80.675) (layer Edge.Cuts) (width 0.15))
   (gr_line (start 60.9 78.743143) (end 98.1 73.35) (layer Edge.Cuts) (width 0.15))
   (gr_line (start 60.05 135.6) (end 60.05 79.6) (layer Edge.Cuts) (width 0.15))
-  (zone (net 1) (net_name GND) (layer B.Cu) (hatch edge 0.508)
-    (connect_pads (clearance 0.3))
+  (zone (net 1) (net_name GND) (layer F.Cu) (hatch edge 0.508)
+    (connect_pads (clearance 0.508))
     (min_thickness 0.254)
-    (fill yes (arc_segments 16) (thermal_gap 0.508) (thermal_bridge_width 0.508))
+    (fill yes (arc_segments 32) (thermal_gap 0.508) (thermal_bridge_width 0.508))
     (polygon
       (pts
-        (xy 58.5 78.1) (xy 58.55 137.1) (xy 117.2 137.1) (xy 136.5 140.8) (xy 140 121)
-        (xy 135.9 120.2) (xy 135.9 76.5) (xy 116.8 72.4) (xy 97.6 72.4)
+        (xy 58.125 76.75) (xy 58.45 138.925) (xy 116.625 139.275) (xy 155.275 150.7) (xy 165.7 126)
+        (xy 157.475 122.975) (xy 158.8 77.425) (xy 112.425 69) (xy 94.775 70.35) (xy 62.625 75.575)
       )
     )
   )
-  (zone (net 1) (net_name GND) (layer F.Cu) (hatch edge 0.508)
-    (connect_pads (clearance 0.3))
+  (zone (net 1) (net_name GND) (layer B.Cu) (hatch edge 0.508)
+    (connect_pads (clearance 0.508))
     (min_thickness 0.254)
-    (fill yes (arc_segments 16) (thermal_gap 0.508) (thermal_bridge_width 0.508))
+    (fill yes (arc_segments 32) (thermal_gap 0.508) (thermal_bridge_width 0.508))
     (polygon
       (pts
-        (xy 58.55 78.1) (xy 58.55 137.1) (xy 117.2 137.1) (xy 136.5 140.8) (xy 140 121)
-        (xy 135.9 120.2) (xy 135.9 76.5) (xy 116.9 72.4) (xy 97.6 72.4)
+        (xy 58.125 76.8) (xy 58.45 138.85) (xy 116.65 139.25) (xy 155.3 150.7) (xy 165.7 126)
+        (xy 157.5 122.95) (xy 158.8 77.425) (xy 112.4 69) (xy 94.75 70.35) (xy 62.525 75.575)
       )
     )
