File: top-plate&cover-plate/Pinky2-top-plate.kicad_pcb (KiCad board)
At the start: 2 copper layers, 75.3 x 68.3 mm, 7 parts

Commit message: top plate
Parts:
- removed the REF** at (107.8, 122.5)
- removed the REF** at (107.8, 116.3)
- added ?: , , F.Cu at (66.4, 122.5)
- added ?: , , F.Cu at (67.0, 122.3)
- added REF**: breakaway-mousebites, lib:breakaway-mousebites, F.Cu at (108.3, 123.0)
- added REF**: breakaway-mousebites, lib:breakaway-mousebites, F.Cu at (108.3, 116.2)
- moved Ref** 20.8 mm to (134.4, 116.0)
- moved Ref** 19.5 mm to (135.1, 95.7)
- moved HOLE_M2 0.86 mm to (118.6, 139.8)
- moved HOLE_M2 0.86 mm to (118.6, 125.3)
Other:
- board size 75.3 x 68.3 mm -> 94.2 x 68.7 mm

Commit message: design finished
Parts:
- removed ? (x2): , 
Changed lines of the file:
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@@
   (general
     (thickness 1.6)
-    (drawings 71)
+    (drawings 72)
     (tracks 0)
     (zones 0)
-    (modules 9)
+    (modules 7)
     (nets 2)
   )
@@
   (title_block
     (title "Pinky2 top plate")
-    (date 2019-10-06)
+    (date 2019-10-09)
     (rev 1.0)
     (company @tamanishi)
@@
       (clearance 0.85))
   )
-  (module "" (layer F.Cu)
-    (at 66.4 122.5)
-    (fp_text reference "" (at 68.2 123.525) (layer F.SilkS)
-      (effects (font (size 1.27 1.27) (thickness 0.15)))
-    )
-    (fp_text value "" (at 68.2 123.525) (layer F.SilkS)
-      (effects (font (size 1.27 1.27) (thickness 0.15)))
-    )
-    (fp_text user GND (at 71.1305 119.9255) (layer F.SilkS)
-      (effects (font (size 0.75 0.5) (thickness 0.125)))
-    )
-  )
-  (module "" (layer F.Cu)
-    (at 67.05 122.275)
-    (fp_text reference "" (at 68.2 123.525) (layer F.SilkS)
-      (effects (font (size 1.27 1.27) (thickness 0.15)))
-    )
-    (fp_text value "" (at 68.2 123.525) (layer F.SilkS)
-      (effects (font (size 1.27 1.27) (thickness 0.15)))
-    )
-    (fp_text user GND (at 71.1305 119.9255) (layer F.SilkS)
-      (effects (font (size 0.75 0.5) (thickness 0.125)))
-    )
-  )
   (module kbd:HOLE_M2 (layer F.Cu)
     (at 118.58 125.28)
@@
     (pad "" np_thru_hole circle (at 0 0) (size 2.2 2.2) (drill 2.2) (layers *.Cu *.Mask F.SilkS)
       (clearance 0.85))
+  )
+  (dimension 68.78 (width 0.3) (layer F.CrtYd)
+    (gr_text "68.780 mm" (at 50.95 107.74 90) (layer F.CrtYd)
+      (effects (font (size 1.5 1.5) (thickness 0.3)))
+    )
+    (feature1 (pts (xy 56.01 73.35) (xy 52.463579 73.35)))
+    (feature2 (pts (xy 56.01 142.13) (xy 52.463579 142.13)))
+    (crossbar (pts (xy 53.05 142.13) (xy 53.05 73.35)))
+    (arrow1a (pts (xy 53.05 73.35) (xy 53.636421 74.476504)))
+    (arrow1b (pts (xy 53.05 73.35) (xy 52.463579 74.476504)))
+    (arrow2a (pts (xy 53.05 142.13) (xy 53.636421 141.003496)))
+    (arrow2b (pts (xy 53.05 142.13) (xy 52.463579 141.003496)))
   )
   (gr_arc (start 82.849929 123.649995) (end 82.849929 122.949995) (angle -90.81845546) (layer Edge.Cuts) (width 0.15))
@@
   (gr_line (start 60.75 116.175) (end 104.62 116.175) (layer Edge.Cuts) (width 0.15))
   (gr_line (start 154.25 81.468823) (end 154.25 117.35) (layer Edge.Cuts) (width 0.15))
-  (dimension 99.975 (width 0.3) (layer F.CrtYd)
-    (gr_text "99.975 mm" (at 110.0375 68.675) (layer F.CrtYd)
+  (dimension 94.32 (width 0.3) (layer F.CrtYd)
+    (gr_text "94.320 mm" (at 107.21 68.41) (layer F.CrtYd)
       (effects (font (size 1.5 1.5) (thickness 0.3)))
     )
-    (feature1 (pts (xy 160.025 73.4) (xy 160.025 70.188579)))
-    (feature2 (pts (xy 60.05 73.4) (xy 60.05 70.188579)))
-    (crossbar (pts (xy 60.05 70.775) (xy 160.025 70.775)))
-    (arrow1a (pts (xy 160.025 70.775) (xy 158.898496 71.361421)))
-    (arrow1b (pts (xy 160.025 70.775) (xy 158.898496 70.188579)))
-    (arrow2a (pts (xy 60.05 70.775) (xy 61.176504 71.361421)))
-    (arrow2b (pts (xy 60.05 70.775) (xy 61.176504 70.188579)))
+    (feature1 (pts (xy 154.37 73.4) (xy 154.37 69.923579)))
+    (feature2 (pts (xy 60.05 73.4) (xy 60.05 69.923579)))
+    (crossbar (pts (xy 60.05 70.51) (xy 154.37 70.51)))
+    (arrow1a (pts (xy 154.37 70.51) (xy 153.243496 71.096421)))
+    (arrow1b (pts (xy 154.37 70.51) (xy 153.243496 69.923579)))
+    (arrow2a (pts (xy 60.05 70.51) (xy 61.176504 71.096421)))
+    (arrow2b (pts (xy 60.05 70.51) (xy 61.176504 69.923579)))
   )
   (gr_line (start 98.1 73.35) (end 116.2 73.35) (layer Edge.Cuts) (width 0.15))
